Commit message: testing controller setup

File: examples/flexiv_description/flexiv_rizon4s_kinematics_zaxis2.urdf (robot description, URDF)
Before this commit: robot rizon4s, 9 links, 8 joints
Joints:
- joint EE: origin xyz=0.000000 0.000000 0.124000 rpy=0.000000000 0.000000000 -3.141592654 -> xyz=0.0 0.0 0.124 rpy=0.0 0.0 -3.141592653589793
- joint joint1: origin xyz=0.000000 0.000000 0.155000 rpy=0.000000000 -0.000000000 -3.141592654 -> xyz=0.000000 0.000000 0.155000 rpy=0.000000000 -0.000000000 3.141592653
- joint joint2: origin xyz=0.000000 0.030000 0.210000 rpy=-1.570796327 -0.000000000 0.000000000 -> xyz=0.000000 0.030000 0.210000 rpy=-0.000000001 -0.000000000 0.000000000
- joint joint4: origin xyz=-0.020000 -0.030000 0.190000 rpy=-1.570796327 -0.000000000 -3.141592654 -> xyz=-0.020000 -0.030000 0.190000 rpy=-0.000000001 -0.000000000 3.141592653
- joint joint5: origin xyz=-0.020000 0.025000 0.195000 rpy=0.000000000 -0.000000000 -3.141592654 -> xyz=-0.020000 0.025000 0.195000 rpy=0.000000000 -0.000000000 3.141592653
- joint joint6: origin xyz=-0.000000 0.030000 0.190000 rpy=-1.570796327 -0.000000000 -0.000000000 -> xyz=0.000000 0.030000 0.190000 rpy=3.141592653 -0.000000000 0.000000000
- joint joint7: origin xyz=-0.015000 0.073000 0.110000 rpy=-0.000000000 -1.570796306 0.000000000 -> xyz=-0.015 0.073 0.11 rpy=0.0 -1.5707963478683205 0.0
